File: frugal_iot_v02/frugal_iot_v02.kicad_sch (KiCad schematic)
At the start: 63 parts, among them J1 USB-C, J12 J2 SENSORS 6-10, J13 J3 SPARE 6-10, J2 J2 SENSORS 1-5, J3 J3 RS485 1-5, J4 CELL, J5 GPIO10, J6 5V IN (aux), J7 EXT LED, Q1 AO3401A, Q2 AO3401A, SW1 RESET, SW2 BOOT, U1 TP4056, U2 XB5353A, U3 ME6211C33M5G, U4 ESP32-C3-WROOM-02U-N4, U5 SP3485EN

Commit message: V0.2 revision 4: files as ordered from JLCPCB
- J4 (JST-PH cell connector) and J6 (5 V screw terminal) fitted (D34);
  schematic notes, BOM, cost estimate and READMEs updated.
- CPL corrected to JLCPCB's part models (D35): rotation fixes for SOT-23,
  SOT-23-5, SOIC-8 and J4, a separate fix for U2 (XB5353A), and connector
  positions at the centre of each pin row.
- claude-tools scripts find their own location instead of the old
  frugal-layout path; pin1.py added for checking JLCPCB's preview.

Co-Authored-By: Claude Opus 5.5 <noreply@anthropic.com>
Claude-Session: https://claude.ai/code/session_01BQeMed5VuFdLpBSsKxvFwD
Parts:
- J4, J6: now fitted
Other:
- note added: "PROG: I = 1200 / R. 4.7k = 255 mA (default); bridge JP1 (2.35k) = 510 mA (D8). TEMP grounded: no cell thermistor. J4 (JST-PH, fitted from D34): pin 1 = cell -, pin 2 = cell +. Not all JST-PH cells are wired the same way: check polarity (D11). XB5353A (D12) sits in the cell's negative lead: board GND is the pack's P-. Trips at 4.30 V / 2.4 V, 3 A discharge; C3 at its VDD pin."
- note added: "USB-C sink, 5 V only: CC1/CC2 5.1k to GND. D+/D- go straight to the C3's native USB (GPIO19/GPIO18): no USB-UART chip and no ESD chip (D9). J6: XY308-2P screw terminal for external 5 V, e.g. a solar panel (D10; fitted from D34)."
- note removed: "PROG: I = 1200 / R. 4.7k = 255 mA (default); bridge JP1 (2.35k) = 510 mA (D8). TEMP grounded: no cell thermistor. J4 (not fitted, JST-PH footprint): pin 1 = cell -, pin 2 = cell +; solder leads or fit a connector by hand (D11). Check cell polarity. XB5353A (D12) sits in the cell's negative lead: board GND is the pack's P-. Trips at 4.30 V / 2.4 V, 3 A discharge; C3 at its VDD pin."
- note removed: "USB-C sink, 5 V only: CC1/CC2 5.1k to GND. D+/D- go straight to the C3's native USB (GPIO19/GPIO18): no USB-UART chip and no ESD chip (D9). J6 (not fitted): 2.54 mm holes for external 5 V or a hand-soldered XY308-2P (D10)."
Changed lines of the file:
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@@
 	(title_block
 		(title "Frugal-IoT V0.2")
-		(date "2026-10-22")
+		(date "2026-10-28")
 		(rev "0.2")
 		(company "Natural Innovation")
@@
 		)
 	)
-	(text "USB-C sink, 5 V only: CC1/CC2 5.1k to GND. D+/D- go straight to the C3's native USB\n(GPIO19/GPIO18): no USB-UART chip and no ESD chip (D9).\nJ6 (not fitted): 2.54 mm holes for external 5 V or a hand-soldered XY308-2P (D10)."
-		(exclude_from_sim no)
-		(at 33.02 153.67 0)
-		(effects
-			(font
-				(size 1 1)
-			)
-			(justify left)
-		)
-	)
 	(text "ESP32-C3-WROOM-02U MODULE"
 		(exclude_from_sim no)
@@
 		)
 	)
+	(text "USB-C sink, 5 V only: CC1/CC2 5.1k to GND. D+/D- go straight to the C3's native USB\n(GPIO19/GPIO18): no USB-UART chip and no ESD chip (D9).\nJ6: XY308-2P screw terminal for external 5 V, e.g. a solar panel (D10; fitted from D34)."
+		(exclude_from_sim no)
+		(at 33.02 153.67 0)
+		(effects
+			(font
+				(size 1 1)
+			)
+			(justify left)
+		)
+	)
 	(text "SYSTEM POWER: LOAD SHARING, 3.3 V LDO, SWITCHED SENSOR RAIL"
 		(exclude_from_sim no)
@@
 		)
 	)
-	(text "PROG: I = 1200 / R. 4.7k = 255 mA (default); bridge JP1 (2.35k) = 510 mA (D8).\nTEMP grounded: no cell thermistor. J4 (not fitted, JST-PH footprint): pin 1 = cell -,\npin 2 = cell +; solder leads or fit a connector by hand (D11). Check cell polarity.\nXB5353A (D12) sits in the cell's negative lead: board GND is the pack's P-.\nTrips at 4.30 V / 2.4 V, 3 A discharge; C3 at its VDD pin."
+	(text "PROG: I = 1200 / R. 4.7k = 255 mA (default); bridge JP1 (2.35k) = 510 mA (D8).\nTEMP grounded: no cell thermistor. J4 (JST-PH, fitted from D34): pin 1 = cell -,\npin 2 = cell +. Not all JST-PH cells are wired the same way: check polarity (D11).\nXB5353A (D12) sits in the cell's negative lead: board GND is the pack's P-.\nTrips at 4.30 V / 2.4 V, 3 A discharge; C3 at its VDD pin."
 		(exclude_from_sim no)
 		(at 162.56 74.93 0)
@@
 		(on_board yes)
 		(in_pos_files yes)
-		(dnp yes)
+		(dnp no)
 		(property "Reference" "J6"
 			(at 121.92 123.95 0)
@@
 		(on_board yes)
 		(in_pos_files yes)
-		(dnp yes)
+		(dnp no)
 		(property "Reference" "J4"
 			(at 281.305 101.217 0)
